Commit message: change path

File: urdf/bazu_Joint_trajectory_controller.urdf (robot description, URDF)
Before this commit: robot bazu, 8 links, 7 joints
Links:
- link base: geometry collision mesh filename=/home/sangkkim/turtlebot3_ws/src/bazu/meshes/base.stl; visual mesh filename=/home/sangkkim/turtlebot3_ws/src/bazu/meshes/base.stl
- link link_1: geometry collision mesh filename=/home/sangkkim/turtlebot3_ws/src/bazu/meshes/joint_1.stl; visual mesh filename=/home/sangkkim/turtlebot3_ws/src/bazu/meshes/joint_1.stl
- link link_2: geometry collision mesh filename=/home/sangkkim/turtlebot3_ws/src/bazu/meshes/joint_2.stl; visual mesh filename=/home/sangkkim/turtlebot3_ws/src/bazu/meshes/joint_2.stl
- link link_3: geometry collision mesh filename=/home/sangkkim/turtlebot3_ws/src/bazu/meshes/joint_3.stl; visual mesh filename=/home/sangkkim/turtlebot3_ws/src/bazu/meshes/joint_3.stl
- link link_4: geometry collision mesh filename=/home/sangkkim/turtlebot3_ws/src/bazu/meshes/joint_4.stl; visual mesh filename=/home/sangkkim/turtlebot3_ws/src/bazu/meshes/joint_4.stl
- link link_5: geometry collision mesh filename=/home/sangkkim/turtlebot3_ws/src/bazu/meshes/joint_5.stl; visual mesh filename=/home/sangkkim/turtlebot3_ws/src/bazu/meshes/joint_5.stl
- link link_6: geometry collision mesh filename=/home/sangkkim/turtlebot3_ws/src/bazu/meshes/joint_6.stl; visual mesh filename=/home/sangkkim/turtlebot3_ws/src/bazu/meshes/joint_6.stl

File: urdf/bazu_gazebo.urdf (robot description, URDF)
Before this commit: robot bazu, 8 links, 7 joints
Links:
- link base: geometry collision mesh filename=/home/sangkkim/turtlebot3_ws/src/bazu/meshes/base.stl; visual mesh filename=/home/sangkkim/turtlebot3_ws/src/bazu/meshes/base.stl
- link link_1: geometry collision mesh filename=/home/sangkkim/turtlebot3_ws/src/bazu/meshes/joint_1.stl; visual mesh filename=/home/sangkkim/turtlebot3_ws/src/bazu/meshes/joint_1.stl
- link link_2: geometry collision mesh filename=/home/sangkkim/turtlebot3_ws/src/bazu/meshes/joint_2.stl; visual mesh filename=/home/sangkkim/turtlebot3_ws/src/bazu/meshes/joint_2.stl
- link link_3: geometry collision mesh filename=/home/sangkkim/turtlebot3_ws/src/bazu/meshes/joint_3.stl; visual mesh filename=/home/sangkkim/turtlebot3_ws/src/bazu/meshes/joint_3.stl
- link link_4: geometry collision mesh filename=/home/sangkkim/turtlebot3_ws/src/bazu/meshes/joint_4.stl; visual mesh filename=/home/sangkkim/turtlebot3_ws/src/bazu/meshes/joint_4.stl
- link link_5: geometry collision mesh filename=/home/sangkkim/turtlebot3_ws/src/bazu/meshes/joint_5.stl; visual mesh filename=/home/sangkkim/turtlebot3_ws/src/bazu/meshes/joint_5.stl
- link link_6: geometry collision mesh filename=/home/sangkkim/turtlebot3_ws/src/bazu/meshes/joint_6.stl; visual mesh filename=/home/sangkkim/turtlebot3_ws/src/bazu/meshes/joint_6.stl
